File: pcb/BSPD.kicad_sch (KiCad schematic)
At the start: 74 parts, among them J1 Conn_02x06_Counter_Clockwise, Q1 AO3400A, U1 MCP1703A-5002_SOT23, U2 LM339, U3 LM339, U4 74HC32, U5 74HC02

Commit message: Schematic/layout for new revision
Parts:
- removed C1: 100uF, Capacitor_SMD:C_1206_3216Metric, symbol Device:C_Small
- removed C2, C6: 10uF, Capacitor_SMD:C_0805_2012Metric, symbol Device:C_Small
- removed C5: 0.1uF, Capacitor_SMD:C_0402_1005Metric, symbol Device:C_Small
- removed D1: D_Schottky, Diode_SMD:D_SOD-323, symbol Device:D_Schottky
- removed TP1, TP10, TP11, TP12, TP2, TP6, TP7, TP8: Value Pre-Delay, symbol Connector:TestPoint
- removed TP13: Value Post-Delay, symbol Connector:TestPoint
- removed TP14: Sensor Post-Delay, symbol Connector:TestPoint
- removed TP3: Value Error, symbol Connector:TestPoint
- removed TP4: BSE Error, symbol Connector:TestPoint
- removed TP5: TPS Error, symbol Connector:TestPoint
- removed TP9: Sensor Pre-Delay, symbol Connector:TestPoint
- removed U1: MCP1703A-5002_SOT23, Package_TO_SOT_SMD:SOT-23, symbol Regulator_Linear:MCP1703A-5002_SOT23
- added J1: Test header, Connector_PinHeader_2.54mm:PinHeader_2x14_P2.54mm_Vertical, symbol Connector_Generic:Conn_02x14_Odd_Even
- added R5, R6, R7, R8: 1k, Resistor_SMD:R_0402_1005Metric, symbol Device:R_Small
- renumbered C3 to C1, C14 to C10, C15 to C11, C4 to C2, C7 to C3, C8 to C4, C9 to C5, C10 to C6, C11 to C7, C12 to C8, C13 to C9, D2 to D1, D3 to D2, D4 to D3, D5 to D4, D6 to D5, J1 to J2, R6 to R10, R7 to R11, R8 to R12, R9 to R13, R10 to R14, R11 to R15, R12 to R16, R13 to R17, R14 to R18, R15 to R19, R16 to R20, R17 to R21, R18 to R22, R19 to R23, R20 to R24, R21 to R25, R22 to R26, R23 to R27, R5 to R9, U2 to U1, U3 to U2, U4 to U3, U5 to U4
Connections:
- net +5V: now also J1.1 (Pin_1); no longer J2.4 (Pin_4)
- net FAULT_5V: now also J1.27 (Pin_27), R8.2; no longer J2.11 (Pin_11)
- net GND: now also J1.10 (Pin_10), J1.12 (Pin_12), J1.14 (Pin_14), J1.16 (Pin_16), J1.18 (Pin_18), J1.2 (Pin_2), J1.20 (Pin_20), J1.22 (Pin_22), J1.24 (Pin_24), J1.26 (Pin_26), J1.28 (Pin_28), J1.4 (Pin_4), J1.6 (Pin_6), J1.8 (Pin_8)
- net Post-Delay: now also J1.25 (Pin_25)
- net Sensor Error: now also J1.13 (Pin_13), R6.2; no longer J2.2 (Pin_2)
- net Sensor Post-Delay: now also J1.17 (Pin_17)
- net Sensor Pre-Delay: now also J1.15 (Pin_15)
- net Startup: now also R5.2; no longer J2.1 (Pin_1)
- net Value Error: now also J1.19 (Pin_19), R7.2; no longer J2.3 (Pin_3)
- net Value Post-Delay: now also J1.23 (Pin_23)
- net Value Pre-Delay: now also J1.21 (Pin_21)
- net Startup timer: now reaches C8.1, R18.2, U4.9
- net Startup timer: now also J1.3 (Pin_3)
- net Startup button: now reaches C7.1, R17.2, U4.8
- net Startup button: now also J1.5 (Pin_5)
- net BSE Error: now reaches U3.3, U3.9
- net BSE Error: now also J1.9 (Pin_9)
- net Startup post-delay: now reaches U4.10, U4.6
- net Startup post-delay: now also J1.7 (Pin_7)
- net TPS Error: now reaches U3.10, U3.6
- net TPS Error: now also J1.11 (Pin_11)
- new net: J2.2 (Pin_2), R6.1
- new net: J2.1 (Pin_1), R5.1
- new net: J2.11 (Pin_11), R8.1
- new net: J2.3 (Pin_3), R7.1
- new net +5VE: J2.4 (Pin_4)
Other:
- added sheet Power supply (power.kicad_sch)
- note added: "Note: A weak pulldown is provided through the 5v to 3.3v resistor netowrk"
- note removed: "5V Power supply"
- moved on the sheet: C3, C4, D1, J2, RV1, RV2, RV3, RV4, RV5, RV6, RV7, RV8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
