File: pcb/BSPD.kicad_sch (KiCad schematic)
At the start: 42 parts, among them J1 Test header, J2 T4142012121-000, Q1 AO3400A, U1 LM339, U2 LM339, U3 74HC32, U4 LM339, U8 74HC1G04GV,125

Commit message: REV 8 Init
Parts:
- removed C10: 1uF, Capacitor_SMD:C_0402_1005Metric, symbol Device:C_Small
- removed C6: 0.1uF, Capacitor_SMD:C_0402_1005Metric, symbol Device:C_Small
- removed C9: 10uF, Capacitor_SMD:C_0805_2012Metric, symbol Device:C_Small
- removed R19, R20: 100k, Resistor_SMD:R_0402_1005Metric, symbol Device:R_Small
- removed R23, R24: 10k, Resistor_SMD:R_0402_1005Metric, symbol Device:R_Small
- removed U4: LM339, Package_SO:SOIC-14_3.9x8.7mm_P1.27mm, symbol Comparator:LM339
- added C7: 10uF, Capacitor_SMD:C_0805_2012Metric, symbol Device:C_Small
- added R1: 50k, Resistor_SMD:R_0402_1005Metric, symbol Device:R_Small
- added R16: 10k, Resistor_SMD:R_0402_1005Metric, symbol Device:R_Small
- U8: footprint Package_TO_SOT_SMD:SOT-553 -> libraries:SOT23-5_FAS
Connections:
- net +5V: now also R16.2; no longer U2.9 (+)
- net GND: now also C7.2; no longer U2.8 (-)
- net Post-Delay: now also J1.5 (Pin_5), U2.14, R16.1; no longer J1.25 (Pin_25), U3.11
- net Sensor Error: now also U3.13
- net Value Error: now also J1.7 (Pin_7), U3.12; no longer J1.19 (Pin_19)
- net Sensor Post-Delay: no longer names the net of J1.17 (Pin_17)
- net Sensor Post-Delay: no longer U3.13
- net Sensor Pre-Delay: no longer names the net of J1.15 (Pin_15)
- net Value Post-Delay renamed Pre-Delay
- net Pre-Delay: now also U2.9 (+), C7.1, R1.2; no longer U3.12
- net Value Pre-Delay renamed Error
- net Error: now also U3.11, R1.1
- new net DELAY: U2.8 (-)
- no-connect marks 6 -> 5
Other:
- note added: "Delay Circuit"
- note removed: "Delay Circuits"
- moved on the sheet: U3D, U8

Commit message: Rev 8 MFG artifacts
Parts:
- D2: LCSC C72043 -> C2986059
- D3: value Yellow -> Red; LCSC C72038 -> C2286
- U8: value 74HC1G04GV,125 -> SN74AHC1G04DBVR; footprint libraries:SOT23-5_FAS -> Package_TO_SOT_SMD:SOT-23-5; LCSC (none) -> C7465
Other:
- moved on the sheet: D5, Q1, R16, R21, R25, R26, R27
