File: pcb/BSPD.kicad_pcb (KiCad board)
At the start: 4 copper layers, 45 x 63.7 mm, 62 parts, among them J1 Test header, J2 T4142012121-000, Q1 AO3400A, U1 LM339, U2 LM339, U3 74HC32, U4 LM339, U5 L7805, U6 L7805, U8 74HC1G04GV,125

Commit message: REV 8 Init
Parts:
- removed C10: 1uF, Capacitor_SMD:C_0402_1005Metric
- removed C6: 0.1uF, Capacitor_SMD:C_0402_1005Metric
- removed C9: 10uF, Capacitor_SMD:C_0805_2012Metric
- removed R19, R20: 100k, Resistor_SMD:R_0402_1005Metric
- removed R23, R24: 10k, Resistor_SMD:R_0402_1005Metric
- removed RV7, RV8: 10k, Potentiometer_SMD:Potentiometer_Bourns_TC33X_Vertical
- removed U4: LM339, Package_SO:SOIC-14_3.9x8.7mm_P1.27mm
- added C7: 10uF, Capacitor_SMD:C_0805_2012Metric, F.Cu at (142.6, 109.9)
- added R1: 50k, Resistor_SMD:R_0402_1005Metric, F.Cu at (142.7, 113.0)
- added R16: 10k, Resistor_SMD:R_0402_1005Metric, F.Cu at (119.8, 133.8)
- added RV10: 10k, Potentiometer_SMD:Potentiometer_Bourns_TC33X_Vertical, F.Cu at (119.9, 112.2)
- U8: footprint Package_TO_SOT_SMD:SOT-553 -> libraries:SOT23-5_FAS
- moved C4 0.44 mm to (120.2, 131.0)
Connections:
- J1 pad 15: /Sensor Pre-Delay -> unconnected-(J1-Pin_15-Pad15)
- J1 pad 17: /Sensor Post-Delay -> unconnected-(J1-Pin_17-Pad17)
- J1 pad 19: Value Error -> unconnected-(J1-Pin_19-Pad19)
- J1 pad 21: /Value Pre-Delay -> Error
- J1 pad 23: /Value Post-Delay -> Pre-Delay
- J1 pad 25: Post-Delay -> unconnected-(J1-Pin_25-Pad25)
- J1 pad 5: unconnected-(J1-Pin_5-Pad5) -> Post-Delay
- J1 pad 7: unconnected-(J1-Pin_7-Pad7) -> Value Error
- U2 pad 14: unconnected-(U2-Pad14) -> Post-Delay
- U2 pad 8: GND -> DELAY
- U2 pad 9: +5V -> Pre-Delay
- U3 pad 11: Post-Delay -> Error
- U3 pad 12: /Value Post-Delay -> Value Error
- U3 pad 13: /Sensor Post-Delay -> Sensor Error
Routing:
- net /Value Pre-Delay: track 61.2 -> 0.00 mm, vias 4 -> 0
- net Pre-Delay: track 0.00 -> 60.4 mm, vias 0 -> 3
- net /Sensor Pre-Delay: track 52.8 -> 0.00 mm, vias 1 -> 0
- net /Value Post-Delay: track 47.1 -> 0.00 mm, vias 1 -> 0
- net /Sensor Post-Delay: track 40.8 -> 0.00 mm, vias 1 -> 0
- net Error: track 0.00 -> 37.3 mm, vias 0 -> 1
- net VALUE_DELAY: track 33.7 -> 0.00 mm
- net SENSOR_DELAY: track 32.8 -> 0.00 mm
- net Value Error: track 69.2 -> 88.7 mm, vias 2 -> 1
- net Vin: track 81.3 -> 62.4 mm, vias 7 -> 6
- net GND: track 115.4 -> 98.5 mm, vias 45 -> 39
- net DELAY: track 0.00 -> 9.20 mm
- net +5V: track 53.7 -> 46.0 mm, vias 23 -> 18
- net Post-Delay: track 74.6 -> 68.1 mm, vias 3 -> 1
- net TPS_THRESH: track 52.9 -> 49.0 mm
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Other:
- board text added: "High Low Thresh Thresh-"
- board text added: "R10"
- board text removed: "High Low Thresh Thresh"
- board text removed: "Value Sensor"

Commit message: Rev 8 MFG artifacts
Parts:
- U8: value 74HC1G04GV,125 -> NL17SZ04XV5T2G; footprint libraries:SOT23-5_FAS -> Package_TO_SOT_SMD:SOT-23-5
Routing:
- added copper zone on F.Cu, net GND
Other:
- board text added: "Bronco Racing BSPD Rev. 8"
- board text removed: "Bronco Racing BSPD Rev. 7"

Commit message: Memes and Small Adjustments
Parts:
- added G***: LOGO, LOGO, F.Cu at (100.8, 110.1)
- added G***: LOGO, libraries:ACDC, B.Cu at (95.3, 120.2)
- added G***: LOGO, libraries:ACDC, B.Cu at (102.2, 114.0)
- G***: footprint LOGO -> libraries:Outlet
- moved R1 51.8 mm to (90.9, 113.6)
- moved G*** 51.2 mm to (83.4, 115.7)
- moved C13 50.5 mm to (90.8, 141.7)
- moved D4 50.5 mm to (92.5, 133.5)
- moved R27 50.5 mm to (104.4, 123.3)
- moved C1 50.5 mm to (76.0, 132.6)
- moved C12 50.5 mm to (102.9, 130.9)
- moved C14 50.5 mm to (101.6, 128.7)
- moved C16 50.5 mm to (102.1, 132.7)
- moved C17 50.5 mm to (97.9, 143.0)
- moved C18 50.5 mm to (97.1, 119.1)
- moved C2 50.5 mm to (76.0, 135.1)
- moved C4 50.5 mm to (69.7, 131.6)
- moved C7 50.5 mm to (92.1, 110.5)
- moved D1 50.5 mm to (79.3, 133.9)
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Routing:
- net GND: track 98.5 -> 69.1 mm, vias 39 -> 32
- net DELAY: track 9.20 -> 12.5 mm
- net Error: track 37.3 -> 35.4 mm
- net Pre-Delay: track 60.4 -> 58.6 mm
Other:
- board text added: "+5V x Post-Delay Value Error BSE Error TPS Error Sensor Err x x x Error Pre-Delay x Fault-5V"
- board text added: "BSPD REV"
- board text added: "GOTTA LOVE LISTENING TO"
- board text added: "N. Banasky, M. Afnan, March 2025"
- board text added: "∞"
- board text removed: "+5V Start Timer Start Btn Start Post BSE Error TPS Error Sensor Err Sensor Pre Sensor Post Value Error Value Pre Value Post Post-Delay Fault-5V"
- board text removed: "DIDN'T EVEN KNOW THEY WERE CATHOLIC"
- board text removed: "JUST FOUND OUT THAT ELECTRONS HAVE MASS."
- board text removed: "N. Banasky M. Afnan November 2024"
